File: fob/fob_pcb/fob.brd (EAGLE design)
At the start: 152.4 x 101.6 mm, 22 parts, among them SW1 PUSH_BUTTON, SW2 PUSH_BUTTON, SW3 PUSH_BUTTON, SW4 PUSH_BUTTON

Commit message: Update fob.brd
yep
Routing:
- net V1: track 69.4 -> 80.0 mm
- net S3: track 161.0 -> 159.7 mm
Changed lines of the file:
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@@
 <wire x1="95.35" y1="40.54" x2="95.35" y2="22.82" width="0.254" layer="1"/>
 <wire x1="90.17" y1="45.72" x2="95.35" y2="40.54" width="0.254" layer="1"/>
-<wire x1="10.16" y1="13.97" x2="11.43" y2="13.97" width="0.254" layer="16"/>
 <wire x1="49.53" y1="13.97" x2="55.88" y2="7.62" width="0.254" layer="16"/>
 <wire x1="55.88" y1="7.62" x2="60.96" y2="7.62" width="0.254" layer="16"/>
@@
 <wire x1="92.71" y1="20.32" x2="95.21" y2="22.82" width="0.254" layer="1"/>
 <wire x1="95.21" y1="22.82" x2="95.35" y2="22.82" width="0.254" layer="1"/>
-<wire x1="10.16" y1="13.97" x2="49.53" y2="13.97" width="0.254" layer="16"/>
+<wire x1="49.53" y1="13.97" x2="10.16" y2="13.97" width="0.254" layer="16"/>
 </signal>
 <signal name="S2">
@@
 <wire x1="5.08" y1="31.75" x2="5.08" y2="81.7" width="0.254" layer="16"/>
 <wire x1="5.08" y1="81.7" x2="9.78" y2="86.4" width="0.254" layer="16"/>
-<wire x1="13.08" y1="86.4" x2="13.08" y2="91.4" width="0" layer="19" extent="1-1"/>
+<wire x1="13.08" y1="91.4" x2="8.85" y2="91.4" width="0.1524" layer="1"/>
+<wire x1="8.85" y1="91.4" x2="7.62" y2="90.17" width="0.1524" layer="1"/>
+<wire x1="7.62" y1="90.17" x2="7.62" y2="88.56" width="0.1524" layer="1"/>
+<wire x1="7.62" y1="88.56" x2="9.78" y2="86.4" width="0.1524" layer="1"/>
 </signal>
 <signal name="N$1">
